File: keyt_motherboard_nrf51822/keyt.sch (KiCad schematic (older format))
At the start: 49 parts, among them J1 Conn_01x06, J2 Conn_01x06, J3 Conn_01x06, J4 Conn_01x06, J5 Conn_01x06, J6 Conn_01x06, J7 Conn_01x06, J8 Conn_01x06, U1 E73-2G4M04S1D

Commit message: cleaning up
Parts:
- D1, D10, D11, D12, D13, D14, D15, D16, D17, D18, D19, D2, D20, D21, D22, D23, D24, D25, D26, D27, D28, D29, D3, D30, D31, D32, D33, D34, D35, D4, D5, D6, D7, D8, D9: symbol redox_rev1-rescue:D-redox_rev1-rescue -> keyt-rescue:D-redox_rev1-rescue-redox_rev1-rescue
- U1: symbol keyt:E73-2G4M04S1D -> keyt-rescue:E73-2G4M04S1D-keyt-redox_rev1-rescue
- U_LEFT1: symbol redox_rev1-rescue:Core51822B-core51822b -> keyt-rescue:Core51822B-core51822b-redox_rev1-rescue
Connections:
- net col0: no longer D1.1 (K), D10.1 (K), D11.1 (K), D12.1 (K), D13.1 (K), D14.1 (K), D15.1 (K), D16.1 (K), D17.1 (K), D18.1 (K), D19.1 (K), D2.1 (K), D20.1 (K), D21.1 (K), D22.1 (K), D23.1 (K), D24.1 (K), D25.1 (K), D26.1 (K), D27.1 (K), D28.1 (K), D29.1 (K), D3.1 (K), D30.1 (K), D31.1 (K), D32.1 (K), D33.1 (K), D34.1 (K), D35.1 (K), D4.1 (K), D5.1 (K), D6.1 (K), D7.1 (K), D8.1 (K), D9.1 (K), J2.1 (Pin_1), J3.1 (Pin_1), J4.1 (Pin_1), J5.1 (Pin_1), J6.1 (Pin_1), J7.1 (Pin_1), U1.16 (GPIO/P0.04), U1.17 (GPIO/P0.05), U1.18 (GPIO/P0.06), U1.19 (GPIO/P0.07), U1.20 (GPIO/P0.08), U1.21 (GPIO/P0.09), U1.27 (AIN0/P0.13), U1.28 (AIN0/P0.14), U1.33 (AIN0/P0.17), U1.34 (AIN0/P0.18), U1.35 (AIN0/P0.19), U_LEFT1.18 (P04), U_LEFT1.19 (P05), U_LEFT1.20 (P06), U_LEFT1.21 (P07), U_LEFT1.22 (P08), U_LEFT1.23 (P09), U_LEFT1.27 (P13), U_LEFT1.28 (P14), U_LEFT1.33 (P17), U_LEFT1.34 (P18), U_LEFT1.35 (P19)
- new net col1: J2.1 (Pin_1), U1.21 (GPIO/P0.09), U_LEFT1.23 (P09)
- new net col2: J3.1 (Pin_1), U1.20 (GPIO/P0.08), U_LEFT1.22 (P08)
- new net col3: J4.1 (Pin_1), U1.19 (GPIO/P0.07), U_LEFT1.21 (P07)
- new net col4: J5.1 (Pin_1), U1.18 (GPIO/P0.06), U_LEFT1.20 (P06)
- new net col5: J6.1 (Pin_1), U1.17 (GPIO/P0.05), U_LEFT1.19 (P05)
- new net col6: J7.1 (Pin_1), U1.16 (GPIO/P0.04), U_LEFT1.18 (P04)
- new net row0: D1.1 (K), D2.1 (K), D3.1 (K), D4.1 (K), D5.1 (K), D6.1 (K), D7.1 (K), U1.35 (AIN0/P0.19), U_LEFT1.35 (P19)
- new net row1: D10.1 (K), D11.1 (K), D12.1 (K), D13.1 (K), D14.1 (K), D8.1 (K), D9.1 (K), U1.34 (AIN0/P0.18), U_LEFT1.34 (P18)
- new net row2: D15.1 (K), D16.1 (K), D17.1 (K), D18.1 (K), D19.1 (K), D20.1 (K), D21.1 (K), U1.33 (AIN0/P0.17), U_LEFT1.33 (P17)
- new net row3: D22.1 (K), D23.1 (K), D24.1 (K), D25.1 (K), D26.1 (K), D27.1 (K), D28.1 (K), U1.28 (AIN0/P0.14), U_LEFT1.28 (P14)
- new net row4: D29.1 (K), D30.1 (K), D31.1 (K), D32.1 (K), D33.1 (K), D34.1 (K), D35.1 (K), U1.27 (AIN0/P0.13), U_LEFT1.27 (P13)
Changed lines of the file:
@@
 EESchema Schematic File Version 4
-LIBS:redox_rev1-cache
-EELAYER 26 0
+LIBS:keyt-cache
+EELAYER 30 0
 EELAYER END
 $Descr A4 11693 8268
@@
 $EndDescr
 $Comp
-L redox_rev1-rescue:D-redox_rev1-rescue D1
+L keyt-rescue:D-redox_rev1-rescue-redox_rev1-rescue D1
 U 1 1 5A808D18
 P 750 1150
@@
 	600  1050 600  1150
 $Comp
-L redox_rev1-rescue:D-redox_rev1-rescue D8
+L keyt-rescue:D-redox_rev1-rescue-redox_rev1-rescue D8
 U 1 1 5A809C23
 P 750 2500
@@
 	600  2400 600  2500
 $Comp
-L redox_rev1-rescue:D-redox_rev1-rescue D15
+L keyt-rescue:D-redox_rev1-rescue-redox_rev1-rescue D15
 U 1 1 5A80AB90
 P 750 3850
@@
 	600  3750 600  3850
 $Comp
-L redox_rev1-rescue:D-redox_rev1-rescue D22
+L keyt-rescue:D-redox_rev1-rescue-redox_rev1-rescue D22
 U 1 1 5A80ABF1
 P 750 5300
@@
 	600  5200 600  5300
 $Comp
-L redox_rev1-rescue:D-redox_rev1-rescue D29
+L keyt-rescue:D-redox_rev1-rescue-redox_rev1-rescue D29
 U 1 1 5A80E499
 P 750 6700
@@
 NoConn ~ 6450 6500
 $Comp
-L redox_rev1-rescue:Core51822B-core51822b U_LEFT1
+L keyt-rescue:Core51822B-core51822b-redox_rev1-rescue U_LEFT1
 U 1 1 5B82A707
 P 7900 2300
@@
 Connection ~ 600  1150
 $Comp
-L redox_rev1-rescue:D-redox_rev1-rescue D35
+L keyt-rescue:D-redox_rev1-rescue-redox_rev1-rescue D35
 U 1 1 5A80E4E7
 P 750 7600
@@
 $EndComp
 $Comp
-L redox_rev1-rescue:D-redox_rev1-rescue D34
+L keyt-rescue:D-redox_rev1-rescue-redox_rev1-rescue D34
 U 1 1 5A80E4DA
 P 750 7450
@@
 $EndComp
 $Comp
-L redox_rev1-rescue:D-redox_rev1-rescue D33
+L keyt-rescue:D-redox_rev1-rescue-redox_rev1-rescue D33
 U 1 1 5A80E4CD
 P 750 7300
@@
 $EndComp
 $Comp
-L redox_rev1-rescue:D-redox_rev1-rescue D32
+L keyt-rescue:D-redox_rev1-rescue-redox_rev1-rescue D32
 U 1 1 5A80E4C0
 P 750 7150
@@
 $EndComp
 $Comp
-L redox_rev1-rescue:D-redox_rev1-rescue D31
+L keyt-rescue:D-redox_rev1-rescue-redox_rev1-rescue D31
 U 1 1 5A80E4B3
 P 750 7000
@@
 	600  6700 600  6850
 $Comp
-L redox_rev1-rescue:D-redox_rev1-rescue D30
+L keyt-rescue:D-redox_rev1-rescue-redox_rev1-rescue D30
 U 1 1 5A80E4A6
 P 750 6850
@@
 $EndComp
 $Comp
-L redox_rev1-rescue:D-redox_rev1-rescue D28
+L keyt-rescue:D-redox_rev1-rescue-redox_rev1-rescue D28
 U 1 1 5A80AC3F
 P 750 6200
@@
 $EndComp
 $Comp
-L redox_rev1-rescue:D-redox_rev1-rescue D27
+L keyt-rescue:D-redox_rev1-rescue-redox_rev1-rescue D27
 U 1 1 5A80AC32
 P 750 6050
@@
 $EndComp
 $Comp
-L redox_rev1-rescue:D-redox_rev1-rescue D26
+L keyt-rescue:D-redox_rev1-rescue-redox_rev1-rescue D26
 U 1 1 5A80AC25
 P 750 5900
@@
 $EndComp
 $Comp
-L redox_rev1-rescue:D-redox_rev1-rescue D25
+L keyt-rescue:D-redox_rev1-rescue-redox_rev1-rescue D25
 U 1 1 5A80AC18
 P 750 5750
@@
 $EndComp
 $Comp
-L redox_rev1-rescue:D-redox_rev1-rescue D24
+L keyt-rescue:D-redox_rev1-rescue-redox_rev1-rescue D24
 U 1 1 5A80AC0B
 P 750 5600
@@
 	600  5300 600  5450
 $Comp
-L redox_rev1-rescue:D-redox_rev1-rescue D23
+L keyt-rescue:D-redox_rev1-rescue-redox_rev1-rescue D23
 U 1 1 5A80ABFE
 P 750 5450
@@
 $EndComp
 $Comp
-L redox_rev1-rescue:D-redox_rev1-rescue D21
+L keyt-rescue:D-redox_rev1-rescue-redox_rev1-rescue D21
 U 1 1 5A80ABDE
 P 750 4750
@@
 $EndComp
 $Comp
-L redox_rev1-rescue:D-redox_rev1-rescue D20
+L keyt-rescue:D-redox_rev1-rescue-redox_rev1-rescue D20
 U 1 1 5A80ABD1
 P 750 4600
@@
 $EndComp
 $Comp
-L redox_rev1-rescue:D-redox_rev1-rescue D19
+L keyt-rescue:D-redox_rev1-rescue-redox_rev1-rescue D19
 U 1 1 5A80ABC4
 P 750 4450
@@
 $EndComp
 $Comp
-L redox_rev1-rescue:D-redox_rev1-rescue D18
+L keyt-rescue:D-redox_rev1-rescue-redox_rev1-rescue D18
 U 1 1 5A80ABB7
 P 750 4300
@@
 $EndComp
 $Comp
-L redox_rev1-rescue:D-redox_rev1-rescue D17
+L keyt-rescue:D-redox_rev1-rescue-redox_rev1-rescue D17
 U 1 1 5A80ABAA
 P 750 4150
@@
 	600  3850 600  4000
 $Comp
-L redox_rev1-rescue:D-redox_rev1-rescue D16
+L keyt-rescue:D-redox_rev1-rescue-redox_rev1-rescue D16
 U 1 1 5A80AB9D
 P 750 4000
@@
 $EndComp
 $Comp
-L redox_rev1-rescue:D-redox_rev1-rescue D13
+L keyt-rescue:D-redox_rev1-rescue-redox_rev1-rescue D13
 U 1 1 5A809C64
 P 750 3250
@@
 $EndComp
 $Comp
-L redox_rev1-rescue:D-redox_rev1-rescue D12
+L keyt-rescue:D-redox_rev1-rescue-redox_rev1-rescue D12
 U 1 1 5A809C57
 P 750 3100
@@
 $EndComp
 $Comp
-L redox_rev1-rescue:D-redox_rev1-rescue D11
+L keyt-rescue:D-redox_rev1-rescue-redox_rev1-rescue D11
 U 1 1 5A809C4A
 P 750 2950
@@
 $EndComp
 $Comp
-L redox_rev1-rescue:D-redox_rev1-rescue D10
+L keyt-rescue:D-redox_rev1-rescue-redox_rev1-rescue D10
 U 1 1 5A809C3D
 P 750 2800
@@
 $EndComp
 $Comp
-L redox_rev1-rescue:D-redox_rev1-rescue D9
+L keyt-rescue:D-redox_rev1-rescue-redox_rev1-rescue D9
 U 1 1 5A809C30
 P 750 2650
@@
 $EndComp
 $Comp
-L redox_rev1-rescue:D-redox_rev1-rescue D7
+L keyt-rescue:D-redox_rev1-rescue-redox_rev1-rescue D7
 U 1 1 5A8094AD
 P 750 2050
@@
 $EndComp
 $Comp
-L redox_rev1-rescue:D-redox_rev1-rescue D6
+L keyt-rescue:D-redox_rev1-rescue-redox_rev1-rescue D6
 U 1 1 5A8094A0
 P 750 1900
@@
 $EndComp
 $Comp
-L redox_rev1-rescue:D-redox_rev1-rescue D5
+L keyt-rescue:D-redox_rev1-rescue-redox_rev1-rescue D5
 U 1 1 5A809493
 P 750 1750
@@
 $EndComp
 $Comp
-L redox_rev1-rescue:D-redox_rev1-rescue D4
+L keyt-rescue:D-redox_rev1-rescue-redox_rev1-rescue D4
 U 1 1 5A809209
 P 750 1600
@@
 $EndComp
 $Comp
-L redox_rev1-rescue:D-redox_rev1-rescue D3
+L keyt-rescue:D-redox_rev1-rescue-redox_rev1-rescue D3
 U 1 1 5A8091FC
 P 750 1450
@@
 	600  1150 600  1300
 $Comp
-L redox_rev1-rescue:D-redox_rev1-rescue D2
+L keyt-rescue:D-redox_rev1-rescue-redox_rev1-rescue D2
 U 1 1 5A80908F
 P 750 1300
@@
 	600  3250 600  3400
 $Comp
-L redox_rev1-rescue:D-redox_rev1-rescue D14
+L keyt-rescue:D-redox_rev1-rescue-redox_rev1-rescue D14
 U 1 1 5A809C71
 P 750 3400
@@
 P03
 $Comp
-L keyt:E73-2G4M04S1D U1
+L keyt-rescue:E73-2G4M04S1D-keyt-redox_rev1-rescue U1
 U 1 1 5C733501
 P 9700 4700
@@
 Text GLabel 7900 4850 2    60   Input ~ 0
 P12
-Text GLabel 600  1150 0    60   Input ~ 0
-col0
-Text GLabel 600  2500 0    60   Input ~ 0
-col0
-Text GLabel 600  3850 0    60   Input ~ 0
-col0
-Text GLabel 600  5300 0    60   Input ~ 0
-col0
-Text GLabel 600  6700 0    60   Input ~ 0
-col0
-Text GLabel 600  1300 0    60   Input ~ 0
-col1
-Text GLabel 600  2650 0    60   Input ~ 0
-col1
-Text GLabel 600  4000 0    60   Input ~ 0
-col1
-Text GLabel 600  5450 0    60   Input ~ 0
-col1
-Text GLabel 600  6850 0    60   Input ~ 0
-col1
-Text GLabel 600  1450 0    60   Input ~ 0
-col2
-Text GLabel 600  2800 0    60   Input ~ 0
-col2
-Text GLabel 600  4150 0    60   Input ~ 0
-col2
-Text GLabel 600  5600 0    60   Input ~ 0
-col2
-Text GLabel 600  7000 0    60   Input ~ 0
-col2
-Text GLabel 600  1600 0    60   Input ~ 0
-col3
-Text GLabel 600  2950 0    60   Input ~ 0
-col3
-Text GLabel 600  4300 0    60   Input ~ 0
-col3
-Text GLabel 600  5750 0    60   Input ~ 0
-col3
-Text GLabel 600  7150 0    60   Input ~ 0
-col3
-Text GLabel 600  1750 0    60   Input ~ 0
-col4
-Text GLabel 600  3100 0    60   Input ~ 0
-col4
-Text GLabel 600  4450 0    60   Input ~ 0
-col4
-Text GLabel 600  5900 0    60   Input ~ 0
-col4
-Text GLabel 600  7300 0    60   Input ~ 0
-col4
-Text GLabel 600  1900 0    60   Input ~ 0
-col5
-Text GLabel 600  3250 0    60   Input ~ 0
-col5
-Text GLabel 600  4600 0    60   Input ~ 0
-col5
-Text GLabel 600  6050 0    60   Input ~ 0
-col5
-Text GLabel 600  7450 0    60   Input ~ 0
-col5
-Text GLabel 600  2050 0    60   Input ~ 0
-col6
-Text GLabel 600  3400 0    60   Input ~ 0
-col6
-Text GLabel 600  4750 0    60   Input ~ 0
-col6
-Text GLabel 600  6200 0    60   Input ~ 0
-col6
-Text GLabel 600  7600 0    60   Input ~ 0
-col6
 $EndSCHEMATC
